File: b016_USB_to_ethernet_LAN9500A/board/bridge.sch (KiCad schematic (older format))
At the start: 23 parts, among them U1 LAN9500(A)

Commit message: added part info for silicon parts
Parts:
- added C3, C4: 10pF, Capacitor_SMD:C_0603_1608Metric, symbol Device:C_Small
- added Y1: 25MhZ, Crystal:Crystal_SMD_Abracon_ABM8G-4Pin_3.2x2.5mm, symbol Device:Crystal_GND24_Small
- C1: value C_Small -> 1uF
- C10, C11, C12, C13, C14, C2: value C_Small -> 100nF
- C15, C16, C17, C5, C7, C8: value C_Small -> 4.7nF
- C18, C19, C9: value C_Small -> 1.5nF
- FB2, FB3, FB4: value Ferrite_Bead_Small -> 220R
- U1: MPN (none) -> LAN9500A
Connections:
- net GND: now also C3.2, C4.2, Y1.2, Y1.4
- net at U1.18 (XI): now also C3.1, Y1.3
- net at U1.19 (XO): now also C4.1, Y1.1
Changed lines of the file:
@@
 F 2 "Package_DFN_QFN:QFN-56-1EP_8x8mm_P0.5mm_EP4.5x5.2mm" H 4125 4500 50  0001 C CNN
 F 3 "" H 4125 4500 50  0001 C CNN
+F 4 "LAN9500A" H 4625 4000 50  0001 C CNN "MPN"
 	1    4625 4000
 	1    0    0    -1
@@
 P 4975 2075
 F 0 "FB4" H 5075 2121 50  0000 L CNN
-F 1 "Ferrite_Bead_Small" H 5075 2030 50  0000 L CNN
+F 1 "220R" H 5075 2030 50  0000 L CNN
 F 2 "Inductor_SMD:L_0805_2012Metric" V 4905 2075 50  0001 C CNN
 F 3 "~" H 4975 2075 50  0001 C CNN
@@
 P 5850 2350
 F 0 "C12" H 5942 2396 50  0000 L CNN
-F 1 "C_Small" H 5942 2305 50  0000 L CNN
+F 1 "100nF" H 5942 2305 50  0000 L CNN
 F 2 "Capacitor_SMD:C_0603_1608Metric" H 5850 2350 50  0001 C CNN
 F 3 "~" H 5850 2350 50  0001 C CNN
@@
 P 6250 2350
 F 0 "C14" H 6342 2396 50  0000 L CNN
-F 1 "C_Small" H 6342 2305 50  0000 L CNN
+F 1 "100nF" H 6342 2305 50  0000 L CNN
 F 2 "Capacitor_SMD:C_0603_1608Metric" H 6250 2350 50  0001 C CNN
 F 3 "~" H 6250 2350 50  0001 C CNN
@@
 P 6650 2350
 F 0 "C16" H 6742 2396 50  0000 L CNN
-F 1 "C_Small" H 6742 2305 50  0000 L CNN
+F 1 "4.7nF" H 6742 2305 50  0000 L CNN
 F 2 "Capacitor_SMD:C_0603_1608Metric" H 6650 2350 50  0001 C CNN
 F 3 "~" H 6650 2350 50  0001 C CNN
@@
 P 7050 2350
 F 0 "C18" H 7142 2396 50  0000 L CNN
-F 1 "C_Small" H 7142 2305 50  0000 L CNN
+F 1 "1.5nF" H 7142 2305 50  0000 L CNN
 F 2 "Capacitor_SMD:C_0603_1608Metric" H 7050 2350 50  0001 C CNN
 F 3 "~" H 7050 2350 50  0001 C CNN
@@
 P 5150 1775
 F 0 "C10" H 5242 1821 50  0000 L CNN
-F 1 "C_Small" H 5242 1730 50  0000 L CNN
+F 1 "100nF" H 5242 1730 50  0000 L CNN
 F 2 "Capacitor_SMD:C_0603_1608Metric" H 5150 1775 50  0001 C CNN
 F 3 "~" H 5150 1775 50  0001 C CNN
@@
 P 5550 1775
 F 0 "C11" H 5642 1821 50  0000 L CNN
-F 1 "C_Small" H 5642 1730 50  0000 L CNN
+F 1 "100nF" H 5642 1730 50  0000 L CNN
 F 2 "Capacitor_SMD:C_0603_1608Metric" H 5550 1775 50  0001 C CNN
 F 3 "~" H 5550 1775 50  0001 C CNN
@@
 P 5950 1775
 F 0 "C13" H 6042 1821 50  0000 L CNN
-F 1 "C_Small" H 6042 1730 50  0000 L CNN
+F 1 "100nF" H 6042 1730 50  0000 L CNN
 F 2 "Capacitor_SMD:C_0603_1608Metric" H 5950 1775 50  0001 C CNN
 F 3 "~" H 5950 1775 50  0001 C CNN
@@
 P 6350 1775
 F 0 "C15" H 6442 1821 50  0000 L CNN
-F 1 "C_Small" H 6442 1730 50  0000 L CNN
+F 1 "4.7nF" H 6442 1730 50  0000 L CNN
 F 2 "Capacitor_SMD:C_0603_1608Metric" H 6350 1775 50  0001 C CNN
 F 3 "~" H 6350 1775 50  0001 C CNN
@@
 P 6750 1775
 F 0 "C17" H 6842 1821 50  0000 L CNN
-F 1 "C_Small" H 6842 1730 50  0000 L CNN
+F 1 "4.7nF" H 6842 1730 50  0000 L CNN
 F 2 "Capacitor_SMD:C_0603_1608Metric" H 6750 1775 50  0001 C CNN
 F 3 "~" H 6750 1775 50  0001 C CNN
@@
 P 7150 1775
 F 0 "C19" H 7242 1821 50  0000 L CNN
-F 1 "C_Small" H 7242 1730 50  0000 L CNN
+F 1 "1.5nF" H 7242 1730 50  0000 L CNN
 F 2 "Capacitor_SMD:C_0603_1608Metric" H 7150 1775 50  0001 C CNN
 F 3 "~" H 7150 1775 50  0001 C CNN
@@
 P 2150 1425
 F 0 "C1" H 2242 1471 50  0000 L CNN
-F 1 "C_Small" H 2242 1380 50  0000 L CNN
+F 1 "1uF" H 2242 1380 50  0000 L CNN
 F 2 "Capacitor_SMD:C_0603_1608Metric" H 2150 1425 50  0001 C CNN
 F 3 "~" H 2150 1425 50  0001 C CNN
@@
 P 2550 1425
 F 0 "C2" H 2642 1471 50  0000 L CNN
-F 1 "C_Small" H 2642 1380 50  0000 L CNN
+F 1 "100nF" H 2642 1380 50  0000 L CNN
 F 2 "Capacitor_SMD:C_0603_1608Metric" H 2550 1425 50  0001 C CNN
 F 3 "~" H 2550 1425 50  0001 C CNN
@@
 P 2950 1425
 F 0 "C5" H 3042 1471 50  0000 L CNN
-F 1 "C_Small" H 3042 1380 50  0000 L CNN
+F 1 "4.7nF" H 3042 1380 50  0000 L CNN
 F 2 "Capacitor_SMD:C_0603_1608Metric" H 2950 1425 50  0001 C CNN
 F 3 "~" H 2950 1425 50  0001 C CNN
@@
 P 3350 1425
 F 0 "C9" H 3442 1471 50  0000 L CNN
-F 1 "C_Small" H 3442 1380 50  0000 L CNN
+F 1 "1.5nF" H 3442 1380 50  0000 L CNN
 F 2 "Capacitor_SMD:C_0603_1608Metric" H 3350 1425 50  0001 C CNN
 F 3 "~" H 3350 1425 50  0001 C CNN
@@
 P 3975 1650
 F 0 "FB2" H 4075 1696 50  0000 L CNN
-F 1 "Ferrite_Bead_Small" H 4075 1605 50  0000 L CNN
+F 1 "220R" H 4075 1605 50  0000 L CNN
 F 2 "Inductor_SMD:L_0805_2012Metric" V 3905 1650 50  0001 C CNN
 F 3 "~" H 3975 1650 50  0001 C CNN
@@
 P 4375 1650
 F 0 "FB3" H 4475 1696 50  0000 L CNN
-F 1 "Ferrite_Bead_Small" H 4475 1605 50  0000 L CNN
+F 1 "220R" H 4475 1605 50  0000 L CNN
 F 2 "Inductor_SMD:L_0805_2012Metric" V 4305 1650 50  0001 C CNN
 F 3 "~" H 4375 1650 50  0001 C CNN
@@
 P 3000 1925
 F 0 "C7" H 3092 1971 50  0000 L CNN
-F 1 "C_Small" H 3092 1880 50  0000 L CNN
+F 1 "4.7nF" H 3092 1880 50  0000 L CNN
 F 2 "Capacitor_SMD:C_0603_1608Metric" H 3000 1925 50  0001 C CNN
 F 3 "~" H 3000 1925 50  0001 C CNN
@@
 P 3250 2300
 F 0 "C8" H 3342 2346 50  0000 L CNN
-F 1 "C_Small" H 3342 2255 50  0000 L CNN
+F 1 "4.7nF" H 3342 2255 50  0000 L CNN
 F 2 "Capacitor_SMD:C_0603_1608Metric" H 3250 2300 50  0001 C CNN
 F 3 "~" H 3250 2300 50  0001 C CNN
@@
 Wire Wire Line
 	5950 3050 5725 3050
+$Comp
+L Device:Crystal_GND24_Small Y1
+U 1 1 6044206E
+P 6325 5775
+F 0 "Y1" H 6625 5600 50  0000 R CNN
+F 1 "25MhZ" H 6625 5675 50  0000 R CNN
+F 2 "Crystal:Crystal_SMD_Abracon_ABM8G-4Pin_3.2x2.5mm" H 6325 5775 50  0001 C CNN
+F 3 "~" H 6325 5775 50  0001 C CNN
+F 4 "535-9140-1-ND" H 6325 5775 50  0001 C CNN "MPN"
+	1    6325 5775
+	-1   0    0    1
+$EndComp
+Wire Wire Line
+	6325 6000 6325 5875
+$Comp
+L power:GND #PWR0103
+U 1 1 6044CEE5
+P 6875 6000
+F 0 "#PWR0103" H 6875 5750 50  0001 C CNN
+F 1 "GND" H 6880 5827 50  0000 C CNN
+F 2 "" H 6875 6000 50  0001 C CNN
+F 3 "" H 6875 6000 50  0001 C CNN
+	1    6875 6000
+	1    0    0    -1
+$EndComp
+$Comp
+L power:GND #PWR0104
+U 1 1 6044D547
+P 6325 6000
+F 0 "#PWR0104" H 6325 5750 50  0001 C CNN
+F 1 "GND" H 6330 5827 50  0000 C CNN
+F 2 "" H 6325 6000 50  0001 C CNN
+F 3 "" H 6325 6000 50  0001 C CNN
+	1    6325 6000
+	1    0    0    -1
+$EndComp
+$Comp
+L Device:C_Small C4
+U 1 1 60459F59
+P 6550 5900
+F 0 "C4" H 6642 5946 50  0000 L CNN
+F 1 "10pF" H 6642 5855 50  0000 L CNN
+F 2 "Capacitor_SMD:C_0603_1608Metric" H 6550 5900 50  0001 C CNN
+F 3 "~" H 6550 5900 50  0001 C CNN
+	1    6550 5900
+	1    0    0    -1
+$EndComp
+$Comp
+L power:GND #PWR0106
+U 1 1 604612BF
+P 6550 6000
+F 0 "#PWR0106" H 6550 5750 50  0001 C CNN
+F 1 "GND" H 6555 5827 50  0000 C CNN
+F 2 "" H 6550 6000 50  0001 C CNN
+F 3 "" H 6550 6000 50  0001 C CNN
+	1    6550 6000
+	1    0    0    -1
+$EndComp
+$Comp
+L Device:C_Small C3
+U 1 1 60465D63
+P 5975 5900
+F 0 "C3" H 6067 5946 50  0000 L CNN
+F 1 "10pF" H 6067 5855 50  0000 L CNN
+F 2 "Capacitor_SMD:C_0603_1608Metric" H 5975 5900 50  0001 C CNN
+F 3 "~" H 5975 5900 50  0001 C CNN
+	1    5975 5900
+	1    0    0    -1
+$EndComp
+$Comp
+L power:GND #PWR0109
+U 1 1 60465D6A
+P 5975 6000
+F 0 "#PWR0109" H 5975 5750 50  0001 C CNN
+F 1 "GND" H 5980 5827 50  0000 C CNN
+F 2 "" H 5975 6000 50  0001 C CNN
+F 3 "" H 5975 6000 50  0001 C CNN
+	1    5975 6000
+	1    0    0    -1
+$EndComp
+Wire Wire Line
+	6325 5675 6325 5650
+Wire Wire Line
+	6875 5650 6875 6000
+Wire Wire Line
+	6325 5650 6875 5650
+Wire Wire Line
+	6550 5800 6550 5775
+Connection ~ 6550 5775
+Wire Wire Line
+	6550 5775 6550 5550
+Wire Wire Line
+	6425 5775 6550 5775
+Wire Wire Line
+	5725 5550 6550 5550
+Wire Wire Line
+	5975 5775 6225 5775
+Wire Wire Line
+	5975 5800 5975 5775
+Wire Wire Line
+	5725 5650 5975 5650
+Connection ~ 5975 5775
+Wire Wire Line
+	5975 5775 5975 5650
 $EndSCHEMATC
