File: b017_USB_to_DebugEdge_FT2232/board/bridge.sch (KiCad schematic (older format))
At the start: 29 parts, among them U1 93CxxC, U2 FT2232H, Y1 Crystal_GND24

Commit message: added part info for silicon parts
Parts:
- U1: MPN (none) -> M93C46-WMN6TP
- U2: MPN (none) -> FT2232H
- Y1: value Crystal_GND24 -> 12MhZ; MPN (none) -> NX8045GB-12.000000MHZ
Changed lines of the file:
@@
 F 2 "Package_QFP:LQFP-64_10x10mm_P0.5mm" H 4525 3675 50  0001 C CNN
 F 3 "https://www.ftdichip.com/Support/Documents/DataSheets/ICs/DS_FT2232H.pdf" H 4525 3675 50  0001 C CNN
+F 4 "FT2232H" H 4525 3675 50  0001 C CNN "MPN"
 	1    4525 3675
 	1    0    0    -1
@@
 P 2625 5275
 F 0 "Y1" H 2819 5321 50  0000 L CNN
-F 1 "Crystal_GND24" H 2819 5230 50  0000 L CNN
+F 1 "12MhZ" H 2819 5230 50  0000 L CNN
 F 2 "Crystal:Crystal_SMD_3225-4Pin_3.2x2.5mm" H 2625 5275 50  0001 C CNN
 F 3 "~" H 2625 5275 50  0001 C CNN
+F 4 "NX8045GB-12.000000MHZ" H 2625 5275 50  0001 C CNN "MPN"
 	1    2625 5275
 	1    0    0    -1
@@
 F 2 "Package_SO:SOIC-8_3.9x4.9mm_P1.27mm" H 1400 4575 50  0001 C CNN
 F 3 "http://ww1.microchip.com/downloads/en/DeviceDoc/20001749K.pdf" H 1400 4575 50  0001 C CNN
+F 4 "M93C46-WMN6TP" H 1400 4575 50  0001 C CNN "MPN"
 	1    1400 4575
 	1    0    0    -1
