File: b023_USB_to_16x_ADC_STM32F723IE/board/board.kicad_pcb (KiCad board)
At the start: 4 copper layers, 45 x 61 mm, 42 parts, among them J1 008_USB_2x2, J2 DebugEdge_02x05, J3 003_power_2x2, J4 007_ADC_2x5, J5 007_ADC_2x5, J6 007_ADC_2x5, J7 007_ADC_2x5, U2 STM32F723IEKx, Y1 Crystal 32kHz, Y2 Crystal_GND24

Commit message: improved labeling
Parts:
- added J10: 001_I2C_2x5, on_edge:on_edge_2x05_up_host, F.Cu at (88.1, 81.0)
- added J11: 002_SPI_2x5, on_edge:on_edge_2x05_up_host, F.Cu at (88.0, 113.0)
- added J8: 001_I2C_2x5, on_edge:on_edge_2x05_up_host, F.Cu at (88.0, 129.0)
- added J9: 002_SPI_2x5, on_edge:on_edge_2x05_up_host, F.Cu at (88.0, 97.0)
Connections:
- U2 pad A5: (no net) -> /uC/I2C1_SCL
- U2 pad B4: (no net) -> /uC/I2C1_SDA
- U2 pad C13: (no net) -> /uC/SPI2_MOSI
- U2 pad C14: (no net) -> /uC/SPI2_MISO
- U2 pad D11: (no net) -> /uC/SPI2_SCK
- U2 pad F14: (no net) -> /uC/I2C3_SDA
- U2 pad F15: (no net) -> /uC/I2C3_SCL
- U2 pad K1: (no net) -> /uC/SPI5_SCK
- U2 pad L2: (no net) -> /uC/SPI5_MOSI
- U2 pad L3: (no net) -> /uC/SPI5_MISO
Routing:
- net +5V: track 100.1 -> 187.5 mm, vias 4 -> 7
- net +3V3: track 206.0 -> 244.4 mm, vias 24 -> 25
- net /uC/I2C3_SCL: track 0.00 -> 30.3 mm
- net /uC/I2C3_SDA: track 0.00 -> 29.8 mm
- net /uC/I2C1_SDA: track 0.00 -> 22.9 mm, vias 0 -> 2
- net /uC/SPI5_MISO: track 0.00 -> 21.0 mm, vias 0 -> 2
- net /uC/I2C1_SCL: track 0.00 -> 20.8 mm, vias 0 -> 2
- net /uC/SPI5_MOSI: track 0.00 -> 17.4 mm, vias 0 -> 2
- net /uC/SPI5_SCK: track 0.00 -> 16.8 mm, vias 0 -> 2
- net /uC/SPI2_SCK: track 0.00 -> 15.5 mm
- net /uC/SPI2_MISO: track 0.00 -> 14.5 mm
- net GND: track 298.3 -> 311.3 mm, vias 45 -> 46
- net /uC/SPI2_MOSI: track 0.00 -> 12.7 mm
- net /uC/tdo: track 18.7 -> 20.4 mm
- net /uC/tck: track 20.1 -> 18.4 mm
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- added copper zone on In1.Cu, net GND
