File: b013_ADC_differential_ADS868x/board/board.kicad_pcb (KiCad board)
At the start: 2 copper layers, 21 x 13 mm, 8 parts, among them J1 002_SPI_2x5, J2 007_ADC_2x5, U1 ADS8689RUM

Commit message: changed b013 to use 3.3v as IO voltage and fixed supply voltage bug
Parts:
- added FB1: Ferrite_Bead_Small, Inductor_SMD:L_0603_1608Metric, F.Cu at (136.6, 94.6)
- added R1: 10k, Resistor_SMD:R_0603_1608Metric, F.Cu at (143.8, 87.6)
Connections:
- C5 pad 1: +5V -> +3V3
- U1 pad 14: +5V -> +3V3
Routing:
- net +3V3: track 17.1 -> 40.0 mm, vias 0 -> 2
- net +5V: track 23.4 -> 17.0 mm, vias 1 -> 2
- net Net-(C4-Pad1): track 2.72 -> 4.04 mm
Other:
- board text added: "osf.b013.v0.2"
- board text removed: "osf.b013.v0.1"

Commit message: fixed connectors and power bug
Connections:
- U1 pad 8: Net-(J1-Pad6) -> Net-(J1-Pad2)
- U1 pad 9: Net-(J1-Pad2) -> Net-(J1-Pad6)
Routing:
- net GND: track 35.8 -> 68.3 mm, vias 0 -> 2
- net +3V3: track 40.0 -> 31.8 mm, vias 2 -> 3
- net Net-(J1-Pad6): track 13.4 -> 10.3 mm
- net Net-(J2-Pad3): track 8.52 -> 5.37 mm, vias 1 -> 0
- net Net-(J1-Pad2): track 11.6 -> 13.4 mm
- net Net-(J2-Pad4): track 7.61 -> 8.98 mm, vias 1 -> 2
- net Net-(J1-Pad3): track 9.60 -> 8.54 mm, vias 1 -> 2
- net Net-(J1-Pad4): track 11.5 -> 12.5 mm, vias 1 -> 2
- net Net-(J1-Pad8): track 15.7 -> 16.5 mm
Other:
- board text added: "osf.002.v0.2"
- board text added: "osf.007.v0.2"
- board text removed: "osf.002.v1"
- board text removed: "osf.007.v1"
