File: b024_007_ADC_to_4xDAC_MCP4728/board/board.sch (KiCad schematic (older format))
At the start: 14 parts, among them J1 007_ADC_2x5, J2 001_I2C_2x5, U1 MCP4728

Commit message: updated connectors
Parts:
- J1: symbol put_on_edge:007_ADC_2x5 -> put_on_edge:007_ADC
- J2: symbol put_on_edge:001_I2C_2x5 -> put_on_edge:001_I2C
Connections:
- net at R4.2, U1.2 (SCL): now also J2.4 (SCL); no longer J2.3 (SCL)
- net at R3.2, U1.3 (SDA): now also J2.2 (SDA); no longer J2.4 (SDA)
- no-connect marks 2 -> 3
Changed lines of the file:
@@
 $EndComp
 $Comp
-L put_on_edge:007_ADC_2x5 J1
+L put_on_edge:007_ADC J1
 U 1 1 60349C8B
 P 3450 3750
@@
 	4000 4050 4000 3250
 $Comp
-L put_on_edge:001_I2C_2x5 J2
+L put_on_edge:001_I2C J2
 U 1 1 604040C2
 P 8525 3950
@@
 Wire Wire Line
 	7975 4050 8075 4050
-Wire Wire Line
-	8075 3950 7675 3950
-Wire Wire Line
-	7675 3950 7675 3650
-Wire Wire Line
-	8075 3850 7750 3850
-Wire Wire Line
-	7750 3850 7750 3550
 $Comp
 L power:VCC #PWR0103
@@
 	7350 3450 7350 3650
 Connection ~ 7350 3650
-Wire Wire Line
-	7350 3650 7675 3650
 $Comp
 L Device:C_Small C7
@@
 Wire Wire Line
 	5025 4225 5025 4100
-NoConn ~ 8075 3750
 $Comp
 L power:GND #PWR0120
@@
 	-1   0    0    -1
 $EndComp
+Wire Wire Line
+	8075 3750 7750 3750
+Wire Wire Line
+	7750 3750 7750 3550
+Wire Wire Line
+	7350 3650 8075 3650
+NoConn ~ 8075 3950
+NoConn ~ 8075 3850
 $EndSCHEMATC
