File: b030_STM32F750_breakout/board/uC.sch (KiCad schematic (older format))
At the start: 31 parts, among them U1 STM32F750V8T6-STM32F750V8T6, Y1 Crystal 32kHz, Y2 Crystal_GND24

Commit message: power and ground changed to higherarchial labels in subsheets
Parts:
- C1, C10, C12, C36, C37, C4, C40, C41, C42, C43, C44, C45, C47, C8, C9: symbol Device:C -> Device:C_Small
