File: b020_STM32F745_breakout/pcb/board.sch (KiCad schematic (older format))
At the start: 6 parts, among them J1 003_power_2x2, J2 I2C_2x2, J3 DebugEdge_02x05, J4 006_RMII_2x10, J6 011_GPIO_2x2

Commit message: fixed ground bugs
Parts:
- J1: symbol put_on_edge:003_power_2x2 -> board-rescue:003_power_2x2-put_on_edge
- J2: symbol put_on_edge:001_I2C_2x5 -> board-rescue:001_I2C_2x5-put_on_edge
- J3: symbol Auto-Intern:DebugEdge_02x05 -> board-rescue:DebugEdge_02x05-Auto-Intern
- J4: symbol put_on_edge:006_RMII_2x10 -> board-rescue:006_RMII_2x10-put_on_edge
- J6: symbol put_on_edge:011_GPIO_2x2 -> board-rescue:011_GPIO_2x2-put_on_edge
Changed lines of the file:
@@
 	3425 2300 3425 2500
 $Comp
-L Auto-Intern:DebugEdge_02x05 J3
+L board-rescue:DebugEdge_02x05-Auto-Intern J3
 U 1 1 60225955
 P 3425 2850
@@
 NoConn ~ 4900 2300
 $Comp
-L put_on_edge:001_I2C_2x5 J2
+L board-rescue:001_I2C_2x5-put_on_edge J2
 U 1 1 60256684
 P 3325 6000
@@
 	4650 6100 4900 6100
 $Comp
-L put_on_edge:003_power_2x2 J1
+L board-rescue:003_power_2x2-put_on_edge J1
 U 1 1 6026F0B5
 P 1550 1300
@@
 	1550 1875 1500 1875
 $Comp
-L put_on_edge:006_RMII_2x10 J4
+L board-rescue:006_RMII_2x10-put_on_edge J4
 U 1 1 6030DD15
 P 8375 2800
@@
 NoConn ~ 7925 2750
 $Comp
-L put_on_edge:011_GPIO_2x2 J6
+L board-rescue:011_GPIO_2x2-put_on_edge J6
 U 1 1 6020A5E1
 P 3300 4500
