File: b028_I2C_Host_STM32F042/board/board.kicad_pcb (KiCad board)
At the start: 4 copper layers, 21 x 13 mm, 10 parts, among them J1 DebugEdge_02x05, J2 001_I2C, U6 STM32F042F6Px

Commit message: added stm32f042 breakout
Routing:
- removed copper zone on In1.Cu, net GND
Other:
- copper layers 4 -> 2
