File: b045_1wire_RJ45/board.kicad_pcb (KiCad board)
At the start: 2 copper layers, 21 x 29 mm, 6 parts, among them J1 RJ45, J2 RJ45, J3 005_1wire, U3 TLV74133PDBVR

Commit message: corrected silkscreen
Other:
- board text added: "osf.b045.v0.2"
- board text removed: "osf.b046.v0.1"
