File: b011_PoE_rectifier_LT4321/board/snippet.sch (KiCad schematic (older format))
At the start: 9 parts, among them Q1 PSMN040-100MSEX, Q2 PSMN040-100MSEX, Q3 PSMN040-100MSEX, Q4 PSMN040-100MSEX, Q5 PSMN040-100MSEX, Q6 PSMN040-100MSEX, Q7 PSMN040-100MSEX, Q8 PSMN040-100MSEX, U1 LT4321

Commit message: cleaned up symbol lib paths
Parts:
- U1: symbol Auto-Intern:LT4321 -> board-rescue:LT4321-Auto-Intern
Changed lines of the file:
@@
 	4150 5250 4450 5250
 $Comp
-L Auto-Intern:LT4321 U?
+L board-rescue:LT4321-Auto-Intern U?
 U 1 1 60323155
 P 7150 3850

Commit message: changed mosfet for availability
Parts:
- Q1, Q2, Q3, Q4, Q5, Q6, Q7, Q8: value PSMN040-100MSEX -> TPN3300ANH,LQ; MPN PSMN040-100MSEX -> TPN3300ANH,LQ
Changed lines of the file:
@@
 AR Path="/6031BEFE/603230EE" Ref="Q8"  Part="1"
 F 0 "Q8" V 4350 5125 50  0000 L CNN
-F 1 "PSMN040-100MSEX" V 4675 4500 50  0000 L CNN
+F 1 "TPN3300ANH,LQ" V 4675 4500 50  0000 L CNN
 F 2 "Package_TO_SOT_SMD:LFPAK33" H 4600 5050 50  0001 C CNN
-F 3 "https://assets.nexperia.com/documents/data-sheet/PSMN5R2-60YL.pdf" H 4450 5050 50  0001 C CNN
-F 4 "PSMN040-100MSEX" H 4450 5050 50  0001 C CNN "MPN"
+F 3 "" H 4450 5050 50  0001 C CNN
+F 4 "TPN3300ANH,LQ" H 4450 5050 50  0001 C CNN "MPN"
 	1    4450 5050
 	0    -1   -1   0
@@
 AR Path="/6031BEFE/603230F5" Ref="Q4"  Part="1"
 F 0 "Q4" V 3650 5150 50  0000 L CNN
-F 1 "PSMN040-100MSEX" V 3950 4850 50  0000 L CNN
+F 1 "TPN3300ANH,LQ" V 3950 4850 50  0000 L CNN
 F 2 "Package_TO_SOT_SMD:LFPAK33" H 3875 5050 50  0001 C CNN
-F 3 "https://assets.nexperia.com/documents/data-sheet/PSMN5R2-60YL.pdf" H 3725 5050 50  0001 C CNN
-F 4 "PSMN040-100MSEX" H 3725 5050 50  0001 C CNN "MPN"
+F 3 "" H 3725 5050 50  0001 C CNN
+F 4 "TPN3300ANH,LQ" H 3725 5050 50  0001 C CNN "MPN"
 	1    3725 5050
 	0    -1   -1   0
@@
 AR Path="/6031BEFE/603230FC" Ref="Q7"  Part="1"
 F 0 "Q7" V 4425 4425 50  0000 L CNN
-F 1 "PSMN040-100MSEX" V 4675 3775 50  0000 L CNN
+F 1 "TPN3300ANH,LQ" V 4675 3775 50  0000 L CNN
 F 2 "Package_TO_SOT_SMD:LFPAK33" H 4600 4325 50  0001 C CNN
-F 3 "https://assets.nexperia.com/documents/data-sheet/PSMN5R2-60YL.pdf" H 4450 4325 50  0001 C CNN
-F 4 "PSMN040-100MSEX" H 4450 4325 50  0001 C CNN "MPN"
+F 3 "" H 4450 4325 50  0001 C CNN
+F 4 "TPN3300ANH,LQ" H 4450 4325 50  0001 C CNN "MPN"
 	1    4450 4325
 	0    -1   -1   0
@@
 AR Path="/6031BEFE/60323103" Ref="Q3"  Part="1"
 F 0 "Q3" V 3700 4450 50  0000 L CNN
-F 1 "PSMN040-100MSEX" V 3950 4125 50  0000 L CNN
+F 1 "TPN3300ANH,LQ" V 3950 4125 50  0000 L CNN
 F 2 "Package_TO_SOT_SMD:LFPAK33" H 3875 4325 50  0001 C CNN
-F 3 "https://assets.nexperia.com/documents/data-sheet/PSMN5R2-60YL.pdf" H 3725 4325 50  0001 C CNN
-F 4 "PSMN040-100MSEX" H 3725 4325 50  0001 C CNN "MPN"
+F 3 "" H 3725 4325 50  0001 C CNN
+F 4 "TPN3300ANH,LQ" H 3725 4325 50  0001 C CNN "MPN"
 	1    3725 4325
 	0    -1   -1   0
@@
 AR Path="/6031BEFE/6032310A" Ref="Q6"  Part="1"
 F 0 "Q6" V 4425 3775 50  0000 L CNN
-F 1 "PSMN040-100MSEX" V 4675 3125 50  0000 L CNN
+F 1 "TPN3300ANH,LQ" V 4675 3125 50  0000 L CNN
 F 2 "Package_TO_SOT_SMD:LFPAK33" H 4600 3675 50  0001 C CNN
-F 3 "https://assets.nexperia.com/documents/data-sheet/PSMN5R2-60YL.pdf" H 4450 3675 50  0001 C CNN
-F 4 "PSMN040-100MSEX" H 4450 3675 50  0001 C CNN "MPN"
+F 3 "" H 4450 3675 50  0001 C CNN
+F 4 "TPN3300ANH,LQ" H 4450 3675 50  0001 C CNN "MPN"
 	1    4450 3675
 	0    -1   -1   0
@@
 AR Path="/6031BEFE/60323111" Ref="Q2"  Part="1"
 F 0 "Q2" V 3700 3775 50  0000 L CNN
-F 1 "PSMN040-100MSEX" V 3950 3475 50  0000 L CNN
+F 1 "TPN3300ANH,LQ" V 3950 3475 50  0000 L CNN
 F 2 "Package_TO_SOT_SMD:LFPAK33" H 3875 3675 50  0001 C CNN
-F 3 "https://assets.nexperia.com/documents/data-sheet/PSMN5R2-60YL.pdf" H 3725 3675 50  0001 C CNN
-F 4 "PSMN040-100MSEX" H 3725 3675 50  0001 C CNN "MPN"
+F 3 "" H 3725 3675 50  0001 C CNN
+F 4 "TPN3300ANH,LQ" H 3725 3675 50  0001 C CNN "MPN"
 	1    3725 3675
 	0    -1   -1   0
@@
 AR Path="/6031BEFE/60323118" Ref="Q5"  Part="1"
 F 0 "Q5" V 4425 3075 50  0000 L CNN
-F 1 "PSMN040-100MSEX" V 4675 2450 50  0000 L CNN
+F 1 "TPN3300ANH,LQ" V 4675 2450 50  0000 L CNN
 F 2 "Package_TO_SOT_SMD:LFPAK33" H 4600 2975 50  0001 C CNN
-F 3 "https://assets.nexperia.com/documents/data-sheet/PSMN5R2-60YL.pdf" H 4450 2975 50  0001 C CNN
-F 4 "PSMN040-100MSEX" H 4450 2975 50  0001 C CNN "MPN"
+F 3 "" H 4450 2975 50  0001 C CNN
+F 4 "TPN3300ANH,LQ" H 4450 2975 50  0001 C CNN "MPN"
 	1    4450 2975
 	0    -1   -1   0
@@
 AR Path="/6031BEFE/6032311F" Ref="Q1"  Part="1"
 F 0 "Q1" V 3675 3075 50  0000 L CNN
-F 1 "PSMN040-100MSEX" V 3950 2750 50  0000 L CNN
+F 1 "TPN3300ANH,LQ" V 3950 2750 50  0000 L CNN
 F 2 "Package_TO_SOT_SMD:LFPAK33" H 3875 2975 50  0001 C CNN
-F 3 "https://assets.nexperia.com/documents/data-sheet/PSMN5R2-60YL.pdf" H 3725 2975 50  0001 C CNN
-F 4 "PSMN040-100MSEX" H 3725 2975 50  0001 C CNN "MPN"
+F 3 "" H 3725 2975 50  0001 C CNN
+F 4 "TPN3300ANH,LQ" H 3725 2975 50  0001 C CNN "MPN"
 	1    3725 2975
 	0    -1   -1   0
