File: b014_007_ADC_to_SMA/board/board.sch (KiCad schematic (older format))
At the start: 3 parts, among them J1 Conn_Coaxial, J2 007_ADC_2x2

Commit message: updated analog connector footprint
Parts:
- J2: footprint on_edge:on_edge_2x02_device -> on_edge:on_edge_2x05_device; symbol put_on_edge:007_ADC_2x2 -> put_on_edge:007_ADC
Connections:
- no-connect marks 1 -> 5
Changed lines of the file:
@@
 $EndDescr
 $Comp
-L put_on_edge:007_ADC_2x2 J2
+L put_on_edge:007_ADC J2
 U 1 1 6034B92F
-P 3450 3550
-F 0 "J2" H 3778 3563 50  0000 L CNN
-F 1 "007_ADC_2x2" H 3778 3472 50  0000 L CNN
-F 2 "on_edge:on_edge_2x02_device" H 3750 4200 50  0001 C CNN
-F 3 "" H 3750 4200 50  0001 C CNN
-	1    3450 3550
+P 3450 3750
+F 0 "J2" H 3778 3763 50  0000 L CNN
+F 1 "007_ADC_2x2" H 3778 3672 50  0000 L CNN
+F 2 "on_edge:on_edge_2x05_device" H 3750 4400 50  0001 C CNN
+F 3 "" H 3750 4400 50  0001 C CNN
+	1    3450 3750
 	-1   0    0    -1
 $EndComp
@@
 L power:GND #PWR0112
 U 1 1 6034E58C
-P 3500 4225
-F 0 "#PWR0112" H 3500 3975 50  0001 C CNN
-F 1 "GND" H 3505 4052 50  0000 C CNN
-F 2 "" H 3500 4225 50  0001 C CNN
-F 3 "" H 3500 4225 50  0001 C CNN
-	1    3500 4225
+P 3450 4575
+F 0 "#PWR0112" H 3450 4325 50  0001 C CNN
+F 1 "GND" H 3455 4402 50  0000 C CNN
+F 2 "" H 3450 4575 50  0001 C CNN
+F 3 "" H 3450 4575 50  0001 C CNN
+	1    3450 4575
 	-1   0    0    -1
 $EndComp
 Wire Wire Line
-	3500 4100 3500 4225
+	3450 4450 3450 4575
 $Comp
 L Connector:Conn_Coaxial J1
@@
 Wire Wire Line
 	4300 3825 4575 3825
+NoConn ~ 3900 3750
+NoConn ~ 3900 3850
+NoConn ~ 3900 4050
+NoConn ~ 3900 4150
 $EndSCHEMATC
