File: b078_Ethernet_MAC+PHY_WIZ5500/board/controller.kicad_sch (KiCad schematic)
At the start: 13 parts, among them U1 W5500, Y1 25MHz

Commit message: updated crystal
Parts:
- Y1: DigiKey Part Number CTX1434CT-ND -> CTX1175TR-ND; MPN (none) -> 445I23D25M00000
Changed lines of the file:
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@@
       (effects (font (size 1.27 1.27)) hide)
     )
-    (property "DigiKey Part Number" "CTX1434CT-ND" (id 4) (at 163.83 87.63 90)
+    (property "DigiKey Part Number" "CTX1175TR-ND" (id 4) (at 163.83 87.63 90)
       (effects (font (size 1.27 1.27)) hide)
     )
+    (property "MPN" "445I23D25M00000" (id 5) (at 163.83 87.63 90)
+      (effects (font (size 1.27 1.27)) hide)
+    )
