File: b090_STM32WL55_breakout_LoRa/board/board.kicad_pcb (KiCad board)
At the start: 4 copper layers, 37 x 61.1 mm, 63 parts, among them CN12 SMA-J-P-H-ST-EMI, J1 DebugEdge_02x05, J2 SPI_2x3, J4 UART_2x2, J7 I2C_2x2, J8 UART_2x2, J9 ADC_2x3, U1 BGS13S4N9, U4 NX3L1T3157GM, U6 STM32WL55, X2 32.768KhZ, Y1 12MhZ

Commit message: dev board cloned
Parts:
- removed C1: 3.3pF, Capacitor_SMD:C_0402_1005Metric
- removed C10, C28, C4, C9: 12pF, Capacitor_SMD:C_0603_1608Metric
- removed C3: 1nF, Capacitor_SMD:C_0402_1005Metric
- removed L1: 11nH, Inductor_SMD:L_0402_1005Metric
- removed R1, R12, R13, R3, R9: 10k, Resistor_SMD:R_0603_1608Metric
- removed R10, R11: 100R, Resistor_SMD:R_0402_1005Metric
- removed R2: 1k, Resistor_SMD:R_0603_1608Metric
- removed R5, R6: 2.2k, Resistor_SMD:R_0603_1608Metric
- removed X2: 32.768KhZ, Crystal:Crystal_SMD_3215-2Pin_3.2x1.5mm
- removed Y1: 12MhZ, Crystal:Crystal_SMD_Abracon_ABM8G-4Pin_3.2x2.5mm
- added C17: Capacitor, Capacitor_SMD:C_0402_1005Metric, F.Cu at (140.0, 86.9)
- added C30: ~, Capacitor_SMD:C_0402_1005Metric, F.Cu at (251.4, 93.1)
- added C35: ~, Capacitor_SMD:C_0603_1608Metric, F.Cu at (140.6, 97.9)
- added C37: ~, Capacitor_SMD:C_0402_1005Metric, B.Cu at (138.1, 97.2)
- added C38: ~, Capacitor_SMD:C_0402_1005Metric, F.Cu at (256.0, 95.0)
- added C43: ~, Capacitor_SMD:C_0402_1005Metric, F.Cu at (129.0, 101.9)
- added C44: ~, Capacitor_SMD:C_0402_1005Metric, F.Cu at (129.0, 102.9)
- added C67: , Capacitor_SMD:C_0402_1005Metric, F.Cu at (236.1, 95.2)
- added C73: ~, Capacitor_SMD:C_0402_1005Metric, B.Cu at (133.6, 86.0)
- added C75: ~, Capacitor_SMD:C_0402_1005Metric, F.Cu at (234.6, 84.1)
- added C77: ~, Capacitor_SMD:C_0402_1005Metric, F.Cu at (241.6, 103.5)
- added C78: ~, Capacitor_SMD:C_0402_1005Metric, F.Cu at (244.5, 95.6)
- added C79: ~, Capacitor_SMD:C_0402_1005Metric, F.Cu at (250.3, 95.0)
- added C80: ~, Capacitor_SMD:C_0402_1005Metric, F.Cu at (234.5, 108.2)
- added C81: ~, Capacitor_SMD:C_0402_1005Metric, F.Cu at (237.5, 88.1)
- added C82: ~, Capacitor_SMD:C_0402_1005Metric, F.Cu at (237.4, 108.2)
- added C83: ~, Capacitor_SMD:C_0402_1005Metric, F.Cu at (234.6, 86.1)
- added C84: ~, Capacitor_SMD:C_0402_1005Metric, F.Cu at (237.5, 84.1)
- added C85: ~, Capacitor_SMD:C_0603_1608Metric, B.Cu at (140.6, 97.9)
- added C86: ~, Capacitor_SMD:C_0402_1005Metric, B.Cu at (137.4, 98.2)
- added C87: ~, Capacitor_SMD:C_0603_1608Metric, F.Cu at (231.2, 84.4)
- added C88: ~, Capacitor_SMD:C_0603_1608Metric, F.Cu at (231.2, 86.9)
- added C89: ~, Capacitor_SMD:C_0402_1005Metric, F.Cu at (237.5, 86.1)
- added C93: Capacitor, Capacitor_SMD:C_0402_1005Metric, F.Cu at (245.6, 93.1)
- added C95: Capacitor, Capacitor_SMD:C_0402_1005Metric, F.Cu at (140.5, 90.8)
- added C97: Capacitor, Capacitor_SMD:C_0402_1005Metric, F.Cu at (257.1, 93.1)
- added L11: Inductor, Inductor_SMD:L_0402_1005Metric, F.Cu at (140.0, 89.7)
- added L13: ~, Inductor_SMD:L_0805_2012Metric, B.Cu at (143.4, 97.6)
- added L14: ~, Inductor_SMD:L_0603_1608Metric, F.Cu at (234.8, 77.5)
- added LED1: ~, Diode_SMD:D_0603_1608Metric, F.Cu at (146.5, 93.1)
- added LED2: ~, Diode_SMD:D_0603_1608Metric, F.Cu at (146.5, 91.6)
- added LED3: ~, Diode_SMD:D_0603_1608Metric, F.Cu at (146.5, 94.6)
- added LED4: , MCD_PARTS.PcbLib:LED_0603_VISHAY_VLMS1300-GS08_RED_1A2K_H0P8, F.Cu at (239.1, 114.8)
- added R25: , MCD_PARTS.PcbLib:R0603, F.Cu at (237.7, 114.5)
- added R26: ~, Resistor_SMD:R_0402_1005Metric, F.Cu at (140.5, 91.8)
- added R28: ~, Resistor_SMD:R_0402_1005Metric, B.Cu at (134.9, 87.5)
- added R29: ~, Resistor_SMD:R_0402_1005Metric, B.Cu at (134.0, 87.5)
- added R34: ~, Resistor_SMD:R_0402_1005Metric, F.Cu at (144.0, 94.3)
- added R35: ~, Resistor_SMD:R_0402_1005Metric, F.Cu at (144.0, 92.4)
- added R36: ~, Resistor_SMD:R_0402_1005Metric, F.Cu at (144.0, 93.3)
- added SC1: ~, parts:CLIP_HARWIN_S0951-46R, F.Cu at (142.0, 86.7)
- added SC3: ~, parts:CLIP_HARWIN_S0951-46R, F.Cu at (124.9, 90.3)
- added SC4: ~, parts:CLIP_HARWIN_S0951-46R, F.Cu at (127.0, 81.8)
- added SC5: ~, parts:CLIP_HARWIN_S0951-46R, F.Cu at (124.9, 85.0)
- added SC6: ~, parts:CLIP_HARWIN_S0951-46R, F.Cu at (131.6, 81.8)
- added SC7: ~, parts:CLIP_HARWIN_S0951-46R, F.Cu at (138.4, 81.8)
- added SC8: Shield-clip_S0981-46R, parts:CLIP_HARWIN_S0951-46R_90, F.Cu at (124.9, 98.8)
- added SC9: Shield-clip_S0981-46R, parts:CLIP_HARWIN_S0951-46R_90, F.Cu at (141.9, 98.8)
- added U11: , MCD_PARTS.PcbLib:ESD_ST0201, F.Cu at (236.2, 96.0)
- C11: value 12pF -> Capacitor; footprint Capacitor_SMD:C_0603_1608Metric -> Capacitor_SMD:C_0402_1005Metric
- C12: value 68pF -> Capacitor
- C13, C2, C24, C25: value 33pF -> ~
- C14, C5, C6: value 3.3pF -> ~
- C15: value 2.2pF -> Capacitor
- C16, C19: value 2.7pF -> ~
- C20: value 3.6pF -> ~
- C21: value 5.6pF -> ~
- C22, C7, C92: value 1.2pF -> Capacitor
- C71: value 1nF -> ~
- C72: value 1nF -> ~; moved to B.Cu
- C74: value 47nF -> ~
- C76: value 68pF -> ~
- C8: value 1.3pF -> ~
- CN12: value SMA-J-P-H-ST-EMI -> ~; footprint Connector_Coaxial:SMA_Amphenol_132289_EdgeMount -> parts:CON_SAMTEC_SMA-J-P-X-ST-EM1
- L10: value 3.3nH -> ~
- L2, L4: value 8.7nH -> ~
- L3: value 8.7nH -> Inductor
- L5: value 3.6nH -> Inductor
- L6: value 3nH -> Inductor
- L7: value 33nH -> Inductor
- L8: value 47nH -> ~
- L9: value 0R -> ~
- R27: value 100R -> ~; moved to B.Cu
- U1: value BGS13S4N9 -> ~; footprint parts:PG-TSNP-9-3 -> parts:ICC_TSNP-9-3_1P1X1P1_P040
- U4: value NX3L1T3157GM -> ~; footprint Package_TO_SOT_SMD:SOT-886 -> parts:ICC_SOT886_XSON6
- U6: value STM32WL55 -> ~; footprint Package_DFN_QFN:VQFN-48-1EP_7x7mm_P0.5mm_EP4.1x4.1mm -> parts:ICC_UFBGA73_5X5_P050
- moved C76 120.4 mm to (253.2, 97.0)
- moved C74 112.0 mm to (244.5, 103.4)
- moved C92 109.1 mm to (241.6, 101.5)
- moved C11 27.7 mm to (131.6, 85.2), turned to 90 degrees
- moved C20 7.99 mm to (140.4, 88.3), turned to 90 degrees
- moved L10 4.85 mm to (137.2, 90.4), turned to 90 degrees
- moved C21 4.80 mm to (137.8, 89.0), turned to 0 degrees
- moved U6 4.57 mm to (136.8, 95.3)
- moved C8 4.11 mm to (138.4, 83.8), turned to -90 degrees
- moved L8 4.04 mm to (136.1, 88.2), turned to 90 degrees
- moved C25 3.91 mm to (135.8, 89.6), turned to 180 degrees
- moved C5 3.75 mm to (135.4, 74.2)
- moved C72 3.63 mm to (136.4, 86.3), turned to 0 degrees
- moved L9 3.51 mm to (132.6, 90.0), turned to 90 degrees
- moved L4 3.50 mm to (137.3, 83.8), turned to 90 degrees
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Connections:
- C11 pad 1: Net-(U6-Pad39) -> Net-(C12-Pad1)
- C12 pad 2: Net-(C1-Pad2) -> (no net)
- C14 pad 1: GND -> Net-(C13-Pad1)
- C14 pad 2: Net-(C13-Pad2) -> GND
- C15 pad 1: Net-(C1-Pad2) -> (no net)
- C15 pad 2: Net-(C15-Pad2) -> Net-(C12-Pad1)
- C16 pad 1: Net-(C13-Pad2) -> (no net)
- C16 pad 2: Net-(C16-Pad2) -> Net-(C13-Pad1)
- C19 pad 1: /rf/RFI_N -> (no net)
- C2 pad 1: Net-(C2-Pad1) -> (no net)
- C2 pad 2: Net-(C2-Pad2) -> (no net)
- C20 pad 1: /rf/RFI_P -> (no net)
- C20 pad 2: Net-(C20-Pad2) -> (no net)
- C21 pad 1: GND -> (no net)
- C21 pad 2: Net-(C16-Pad2) -> GND
- C22 pad 1: GND -> (no net)
- C22 pad 2: Net-(C15-Pad2) -> GND
- C24 pad 1: Net-(C24-Pad1) -> GND
- C24 pad 2: GND -> (no net)
- C25 pad 1: Net-(C25-Pad1) -> (no net)
- C5 pad 1: Net-(C5-Pad1) -> (no net)
- C6 pad 1: Net-(C2-Pad2) -> (no net)
- C7 pad 1: GND -> (no net)
- C7 pad 2: Net-(C7-Pad2) -> GND
- C74 pad 1: GND -> (no net)
- C74 pad 2: /rf/VR_PA -> GND
- C76 pad 1: GND -> (no net)
- C76 pad 2: /rf/VR_PA -> GND
- C8 pad 1: GND -> (no net)
- C8 pad 2: Net-(C8-Pad2) -> GND
- C92 pad 1: GND -> (no net)
- C92 pad 2: /rf/VR_PA -> GND
- CN12 pad 1: Net-(C5-Pad1) -> (no net)
- L10 pad 1: Net-(C16-Pad2) -> (no net)
- L10 pad 2: /rf/RFO_LP -> (no net)
- L2 pad 1: Net-(C2-Pad2) -> (no net)
- L2 pad 2: Net-(C5-Pad1) -> (no net)
- L3 pad 1: Net-(C7-Pad2) -> (no net)
- L3 pad 2: Net-(C12-Pad1) -> (no net)
- L4 pad 1: Net-(C8-Pad2) -> Net-(C13-Pad2)
- L4 pad 2: Net-(C13-Pad1) -> (no net)
- L5 pad 1: Net-(C1-Pad2) -> (no net)
- L5 pad 2: Net-(C15-Pad2) -> Net-(C12-Pad1)
- L6 pad 1: Net-(C13-Pad2) -> (no net)
- L6 pad 2: Net-(C16-Pad2) -> Net-(C13-Pad1)
- L7 pad 1: Net-(C15-Pad2) -> (no net)
- L7 pad 2: Net-(C24-Pad1) -> (no net)
- L8 pad 1: Net-(C16-Pad2) -> (no net)
- L8 pad 2: Net-(C25-Pad1) -> (no net)
- L9 pad 1: Net-(C15-Pad2) -> (no net)
- L9 pad 2: /rf/RFO_HP -> (no net)
- R27 pad 1: /rf/FE_CTRL1 -> (no net)
- U1 pad 2: Net-(C8-Pad2) -> (no net)
- U1 pad 3: Net-(C20-Pad2) -> (no net)
- U1 pad 4: Net-(C2-Pad1) -> (no net)
- U1 pad 5: Net-(C7-Pad2) -> (no net)
- U1 pad 7: Net-(C3-Pad1) -> (no net)
- U4 pad 1: Net-(C25-Pad1) -> (no net)
- U4 pad 3: Net-(C24-Pad1) -> (no net)
- U4 pad 4: /rf/VR_PA -> (no net)
- U4 pad 5: /rf/VDD_APP -> (no net)
- U4 pad 6: /rf/FE_CTRL1 -> (no net)
Routing:
- net GND: track 214.0 -> 109.4 mm, vias 16 -> 5
- net (no net): track 0.00 -> 78.5 mm, vias 0 -> 3
- net +5V: track 96.6 -> 32.4 mm, vias 5 -> 4
- net /uC/NRESET: track 54.7 -> 3.73 mm, vias 3 -> 1
- net /UART0_RX: track 51.7 -> 2.12 mm, vias 2 -> 1
- net /UART0_TX: track 49.9 -> 4.08 mm, vias 2 -> 1
- net +3V3: track 144.7 -> 99.0 mm, vias 6 -> 5
- net /ADC1: track 43.3 -> 0.84 mm, vias 2 -> 0
- net /ADC0: track 40.2 -> 0.00 mm, vias 2 -> 0
- net /uC/SPI_SCK: track 39.1 -> 5.05 mm
- net /uC/SPI_MISO: track 38.0 -> 4.64 mm
- net /uC/SPI_MOSI: track 36.9 -> 4.34 mm
- net /ADC2: track 33.9 -> 1.48 mm, vias 2 -> 0
- net /uC/SWO: track 33.4 -> 3.05 mm, vias 1 -> 0
- net /uC/SPI_CS: track 32.6 -> 5.43 mm
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- added copper zone on F.Cu, net (none)
