File: b077_PoE_PD_DCDC_non_isolated_SI3404/board/dcdc.kicad_sch (KiCad schematic)
At the start: 27 parts, among them U1 Si3404

Commit message: fixed missing connections mentioned in PR #64. cleaned up lib connections and bumped version to 1.0
Parts:
- C2: symbol Device:CP_Small -> Device:C_Polarized_Small
- FB1, FB2: symbol Device:Ferrite_Bead_Small -> Device:FerriteBead_Small
Changed lines of the file:
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@@
     (pin "2")
   )
-  (symbol (lib_id "Device:Ferrite_Bead_Small") (at 38.1 97.79 90) (unit 1)
+  (symbol (lib_id "Device:FerriteBead_Small") (at 38.1 97.79 90) (unit 1)
     (in_bom yes) (on_board yes)
     (property "Reference" "FB1" (id 0) (at 38.0619 91.44 90))
@@
     (pin "2")
   )
-  (symbol (lib_id "Device:Ferrite_Bead_Small") (at 38.1 116.84 90) (unit 1)
+  (symbol (lib_id "Device:FerriteBead_Small") (at 38.1 116.84 90) (unit 1)
     (in_bom yes) (on_board yes) (fields_autoplaced)
     (property "Reference" "FB2" (id 0) (at 38.0619 110.49 90))
@@
     (pin "2")
   )
-  (symbol (lib_id "Device:CP_Small") (at 73.66 74.93 0) (unit 1)
+  (symbol (lib_id "Device:C_Polarized_Small") (at 73.66 74.93 0) (unit 1)
     (in_bom yes) (on_board yes)
     (property "Reference" "C2" (id 0) (at 76.2 73.1138 0)

Commit message: Fix supply, better thermal mgmt.
Parts:
- added C?: 100nF, Capacitor_SMD:C_0603_1608Metric, symbol Device:C_Small
- TP1: value TestPoint -> GND2_OUT; footprint (none) -> TestPoint:TestPoint_Pad_D1.0mm
- TP2: value TestPoint -> VT15; footprint (none) -> TestPoint:TestPoint_Pad_D1.0mm; now left out of the parts list
Connections:
- net 5V: now also R3.2, R5.2, U1.13 (VPOS), C?.1
- net GND_IN: now reaches C1.2, FB2.2, R4.1, U1.11 (NC), U1.12 (NC), U1.14 (VNEG), U1.15 (NC), U1.17 (NC), U1.20 (NC), U1.21 (EPAD), U1.7 (NC)
- net GND_IN: now also C?.2
- net GND2_OUT: now reaches D3.2 (A), L1.1, TP1.1, U1.18 (SWO)
Other:
- moved on the sheet: C1, C10, C12, C2, C3, C4, C5, C6, C7, C8, C9, D3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
