File: b076_PoE_PD_DCDC_isolated_SI3404/board/board.kicad_sch (KiCad schematic)
At the start: 2 parts, among them J1 013_PoE_rectified, J2 003_power

Commit message: Update PWR fix
Changed lines of the file:
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@@
   (junction (at 195.58 81.28) (diameter 0) (color 0 0 0 0)
+  )
+  (junction (at 167.64 81.28) (diameter 0) (color 0 0 0 0)
   )
   (no_connect (at 181.61 64.77))
@@
     (stroke (width 0) (type default) (color 0 0 0 0))
   )
+  (wire (pts (xy 52.07 83.82) (xy 62.23 83.82))
+    (stroke (width 0) (type default) (color 0 0 0 0))
+  )
   (wire (pts (xy 105.41 88.9) (xy 105.41 85.09))
     (stroke (width 0) (type default) (color 0 0 0 0))
   )
+  (wire (pts (xy 52.07 81.28) (xy 52.07 83.82))
+    (stroke (width 0) (type default) (color 0 0 0 0))
+  )
   (wire (pts (xy 195.58 78.74) (xy 195.58 81.28))
     (stroke (width 0) (type default) (color 0 0 0 0))
@@
     (stroke (width 0) (type default) (color 0 0 0 0))
   )
+  (wire (pts (xy 167.64 81.28) (xy 187.96 81.28))
+    (stroke (width 0) (type default) (color 0 0 0 0))
+  )
   (wire (pts (xy 80.01 62.23) (xy 113.03 62.23))
     (stroke (width 0) (type default) (color 0 0 0 0))
@@
     (stroke (width 0) (type default) (color 0 0 0 0))
   )
+  (wire (pts (xy 167.64 79.375) (xy 167.64 81.28))
+    (stroke (width 0) (type default) (color 0 0 0 0))
+  )
   (wire (pts (xy 146.05 69.85) (xy 181.61 69.85))
     (stroke (width 0) (type default) (color 0 0 0 0))
   )
-  (wire (pts (xy 146.05 81.28) (xy 187.96 81.28))
+  (wire (pts (xy 146.05 81.28) (xy 167.64 81.28))
     (stroke (width 0) (type default) (color 0 0 0 0))
   )
@@
     )
     (property "Datasheet" "" (id 3) (at 62.23 87.63 0)
+      (effects (font (size 1.27 1.27)) hide)
+    )
+    (pin "1")
+  )
+  (symbol (lib_id "power:PWR_FLAG") (at 52.07 81.28 0) (unit 1)
+    (in_bom yes) (on_board yes) (fields_autoplaced)
+    (property "Reference" "#FLG0102" (id 0) (at 52.07 79.375 0)
+      (effects (font (size 1.27 1.27)) hide)
+    )
+    (property "Value" "PWR_FLAG" (id 1) (at 52.07 76.2 0))
+    (property "Footprint" "" (id 2) (at 52.07 81.28 0)
+      (effects (font (size 1.27 1.27)) hide)
+    )
+    (property "Datasheet" "~" (id 3) (at 52.07 81.28 0)
       (effects (font (size 1.27 1.27)) hide)
     )
@@
     (pin "4")
     (pin "5")
+  )
+  (symbol (lib_id "power:PWR_FLAG") (at 167.64 79.375 0) (unit 1)
+    (in_bom yes) (on_board yes) (fields_autoplaced)
+    (property "Reference" "#FLG0101" (id 0) (at 167.64 77.47 0)
+      (effects (font (size 1.27 1.27)) hide)
+    )
+    (property "Value" "PWR_FLAG" (id 1) (at 167.64 73.66 0))
+    (property "Footprint" "" (id 2) (at 167.64 79.375 0)
+      (effects (font (size 1.27 1.27)) hide)
+    )
+    (property "Datasheet" "~" (id 3) (at 167.64 79.375 0)
+      (effects (font (size 1.27 1.27)) hide)
+    )
+    (pin "1")
   )
   (symbol (lib_id "put_on_edge:003_power") (at 193.04 64.77 0) (unit 1)
@@
   )
   (symbol_instances
+    (path "/bc35d20a-3a1b-48e8-a2f8-83c0dfacde63"
+      (reference "#FLG0101") (unit 1) (value "PWR_FLAG") (footprint "")
+    )
+    (path "/4ebf59df-bc69-439f-b9f2-cb433efbca66"
+      (reference "#FLG0102") (unit 1) (value "PWR_FLAG") (footprint "")
+    )
+    (path "/bd58ad52-36c7-460d-b58d-1e0ca17757a0/0eb913cb-2e9c-477b-b795-6ef7b7345402"
+      (reference "#FLG0103") (unit 1) (value "PWR_FLAG") (footprint "")
+    )
+    (path "/bd58ad52-36c7-460d-b58d-1e0ca17757a0/594e3aa4-35e3-49ed-af28-cea9c66d236f"
+      (reference "#FLG0104") (unit 1) (value "PWR_FLAG") (footprint "")
+    )
+    (path "/bd58ad52-36c7-460d-b58d-1e0ca17757a0/cdb46dee-fa1a-4c10-acbf-d2cfe6276377"
+      (reference "#FLG0105") (unit 1) (value "PWR_FLAG") (footprint "")
+    )
     (path "/00000000-0000-0000-0000-00006044056a"
       (reference "#PWR0101") (unit 1) (value "GND") (footprint "")
@@
       (reference "R15") (unit 1) (value "0R") (footprint "Resistor_SMD:R_0603_1608Metric")
     )
-    (path "/bd58ad52-36c7-460d-b58d-1e0ca17757a0/a00d687c-be70-4f1c-8302-2dfcd4082526"
-      (reference "TP1") (unit 1) (value "TestPoint") (footprint "")
-    )
-    (path "/bd58ad52-36c7-460d-b58d-1e0ca17757a0/bfc65580-ac97-4472-8c25-735a5ff6ac18"
-      (reference "TP2") (unit 1) (value "TestPoint") (footprint "")
-    )
     (path "/bd58ad52-36c7-460d-b58d-1e0ca17757a0/4b66da4e-eb7a-44b8-8c71-817f1bb4a9e1"
