File: b092_TMCS1100/board/vref_amp.kicad_sch (KiCad schematic)
At the start: 7 parts, among them U2 LM4041-N, U3 LMV601

Commit message: added silkscreen, bigger gap between input
Parts:
- C4: value 1uF -> 100nF
Changed lines of the file:
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@@
     (stroke (width 0) (type default) (color 0 0 0 0))
   )
-  (wire (pts (xy 120.65 129.54) (xy 115.57 129.54))
+  (wire (pts (xy 105.41 100.33) (xy 120.65 100.33))
+    (stroke (width 0) (type default) (color 0 0 0 0))
+  )
+  (wire (pts (xy 104.14 129.54) (xy 120.65 129.54))
     (stroke (width 0) (type default) (color 0 0 0 0))
   )
@@
     (stroke (width 0) (type default) (color 0 0 0 0))
   )
-  (wire (pts (xy 115.57 100.33) (xy 120.65 100.33))
-    (stroke (width 0) (type default) (color 0 0 0 0))
-  )
   (wire (pts (xy 120.65 109.22) (xy 135.89 109.22))
     (stroke (width 0) (type default) (color 0 0 0 0))
@@
     (effects (font (size 1.27 1.27)) (justify left bottom))
   )
-  (hierarchical_label "GND" (shape input) (at 115.57 129.54 180)
+  (hierarchical_label "GND" (shape input) (at 104.14 129.54 180)
     (effects (font (size 1.27 1.27)) (justify right))
   )
-  (hierarchical_label "VDD_2.7-5V" (shape input) (at 115.57 100.33 180)
+  (hierarchical_label "VDD_2.7-5V" (shape input) (at 105.41 100.33 180)
     (effects (font (size 1.27 1.27)) (justify right))
   )
@@
     (effects (font (size 1.27 1.27)) (justify right))
   )
-  (symbol (lib_id "Amplifier_Operational:LMV601") (at 166.37 111.76 0) (unit 1)
+  (symbol (lib_id "Amplifier_Operational:LMV601") (at 166.37 111.76 0)
     (in_bom yes) (on_board yes)
     (property "Reference" "U3" (id 0) (at 175.1076 110.5916 0)
@@
     (pin "6")
   )
-  (symbol (lib_id "Device:R_Small") (at 166.37 129.54 90) (unit 1)
+  (symbol (lib_id "Device:R_Small") (at 166.37 129.54 90)
     (in_bom yes) (on_board yes)
     (property "Reference" "R4" (id 0) (at 166.37 134.62 90))
@@
     (pin "2")
   )
-  (symbol (lib_id "Device:R_Small") (at 120.65 104.14 0) (unit 1)
+  (symbol (lib_id "Device:R_Small") (at 120.65 104.14 0)
     (in_bom yes) (on_board yes)
     (property "Reference" "R1" (id 0) (at 115.57 104.14 90))
@@
     (pin "2")
   )
-  (symbol (lib_id "Device:C_Small") (at 120.65 120.65 0) (unit 1)
+  (symbol (lib_id "Device:C_Small") (at 120.65 120.65 0)
     (in_bom yes) (on_board yes)
     (property "Reference" "C4" (id 0) (at 122.9868 119.4816 0)
       (effects (font (size 1.27 1.27)) (justify left))
     )
-    (property "Value" "1uF" (id 1) (at 122.9868 121.793 0)
+    (property "Value" "100nF" (id 1) (at 122.9868 121.793 0)
       (effects (font (size 1.27 1.27)) (justify left))
     )
@@
     (pin "2")
   )
-  (symbol (lib_id "Device:R_Small") (at 142.24 115.57 0) (mirror y) (unit 1)
+  (symbol (lib_id "Device:R_Small") (at 142.24 115.57 0) (mirror y)
     (in_bom yes) (on_board yes)
     (property "Reference" "R2" (id 0) (at 147.32 115.57 90))
@@
     (pin "2")
   )
-  (symbol (lib_id "iso_curr_sns_TCMS1100-rescue:LM4041-N-2021_bt5_headtracker_symbols") (at 135.89 120.65 270) (mirror x) (unit 1)
+  (symbol (lib_id "iso_curr_sns_TCMS1100-rescue:LM4041-N-2021_bt5_headtracker_symbols") (at 135.89 120.65 270) (mirror x)
     (in_bom yes) (on_board yes)
     (property "Reference" "U2" (id 0) (at 133.6548 119.4816 90)
@@
     (pin "3")
   )
-  (symbol (lib_id "Device:R_Small") (at 142.24 125.73 0) (mirror y) (unit 1)
+  (symbol (lib_id "Device:R_Small") (at 142.24 125.73 0) (mirror y)
     (in_bom yes) (on_board yes)
     (property "Reference" "R3" (id 0) (at 147.32 125.73 90))
