File: b096_MAC_ID_chip_11AA02E48_11AA02E64/mac.kicad_sch (KiCad schematic)
At the start: 1 part, among them U1 11AA02E48

Commit message: added exact part number
Parts:
- U1: DigiKey_PN (none) -> 11AA02E48T-I/TTCT-ND; MPN (none) -> 11AA02E48T-I/TT
Changed lines of the file:
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@@
       (effects (font (size 1.27 1.27)) hide)
     )
-    (property "Datasheet" "" (id 3) (at 107.95 106.68 0)
+    (property "Datasheet" "https://ww1.microchip.com/downloads/aemDocuments/documents/OTH/ProductDocuments/DataSheets/11AA02E48-11AA02E64-2K-UNIO-Serial-EEPROMs-Data-Sheet-20002122E.pdf" (id 3) (at 107.95 106.68 0)
       (effects (font (size 1.27 1.27)) hide)
     )
+    (property "DigiKey_PN" "11AA02E48T-I/TTCT-ND" (id 4) (at 107.95 106.68 0)
+      (effects (font (size 1.27 1.27)) hide)
+    )
+    (property "MPN" "11AA02E48T-I/TT" (id 5) (at 107.95 106.68 0)
+      (effects (font (size 1.27 1.27)) hide)
+    )
